Commit message: ros2

File: description/robot.urdf.xacro (robot description, xacro)
@@ -2,3 +2,6 @@
 <robot xmlns:xacro="http://www.ros.org/wiki/xacro"  name="robot_arm">
     <xacro:include filename="robot_core.xacro" />
+    <!-- <xacro:include filename="robot_core_2.xacro" />  -->
+    <xacro:include filename="ros2_control.xacro" />
+    <xacro:include filename="gazebo.xacro" />
 </robot>

File: description/robot_core_2.xacro (robot description, xacro)
@@ -58,5 +58,5 @@
             <origin xyz="0 0 0"/>
             <geometry>
-                <mesh filename="package://example_package/meshes/rot_base.stl" scale="0.01 0.01 0.01" />
+                <mesh filename="package://example_package/meshes/rot_base.stl" scale="0.1 0.1 0.1" />
             </geometry>
         </collision>

Commit message: ros2_control with mesh file

File: description/robot.urdf.xacro (robot description, xacro)
@@ -4,4 +4,3 @@
     <!-- <xacro:include filename="robot_core_2.xacro" />  -->
     <xacro:include filename="ros2_control.xacro" />
-    <xacro:include filename="gazebo.xacro" />
 </robot>

File: description/robot_core.xacro (robot description, xacro)
@@ -41,5 +41,5 @@
     </link>
     <!-- ___________________________________ Rotating Base _______________________________ -->
-    <joint name="rot_base" type="continuous">
+    <joint name="rot_base_joint" type="continuous">
     <parent link="base"/>
     <child link="rot_base"/>
@@ -56,7 +56,7 @@
         </visual>
         <collision>
-            <origin xyz="0 0 0"/>
+            <origin xyz="-0.1355 0 0.2"/>
             <geometry>
-                <mesh filename="package://example_package/meshes/rot_base.stl" scale="0.01 0.01 0.01" />
+                <mesh filename="package://example_package/meshes/rot_base.stl" scale="0.001 0.001 0.001" />
             </geometry>
         </collision>

File: description/ros2_control.xacro (robot description, xacro)
@@ -1,13 +1,27 @@
 <?xml version="1.0"?>
 <robot xmlns:xacro="http://www.ros.org/wiki/xacro">
-    <ros2_control name="gazebo_ros_controller">
+    <ros2_control name="GazeboSystem" type="system">
         <hardware>
-            <plugin>gazebo_ros2_control/GazeboSystemInterface</plugin>
+            <plugin>gazebo_ros2_control/GazeboSystem</plugin>
         </hardware>
         <joint name="rot_base">
             <command_interface name="position"/>
+                <param name="min">-3.14</param>
+                <param name="max">3.14</param>
             <state_interface name="position"/>
             <state_interface name="velocity"/>
         </joint>
     </ros2_control>
+    <gazebo>
+        <plugin name="gazebo_ros2_control" filename="libgazebo_ros2_control.so">
+            <parameters>$(find example_package)/config/controllers.yaml</parameters>
+        </plugin>
+    </gazebo>
+    <gazebo reference="base">
+        <material>Gazebo/White</material>
+    </gazebo>
+    <gazebo reference="rot_base">
+        <material>Gazebo/Blue</material>
+        <dynamics damping="0.1" friction="0.2"/>
+    </gazebo>
 </robot>
